Commit message: changed for RGB-D grasper

File: models/panda_description/panda_grasp.urdf (robot description, URDF)
Before this commit: robot panda, 12 links, 11 joints
Links:
- added link panda_grasp_center, mass 0.0; collision sphere radius=0.0001; visual sphere radius=0.0001
Joints:
- added joint panda_grasp_center_joint: type fixed, parent panda_hand, child panda_grasp_center, origin xyz=0 0 0.1244 rpy=0 0 0
